Commit message: added tcp to urdf model

File: omron_tm12_robotiq_2f_140/urdf/omron_tm12_robotiq_2f_140.urdf.xacro (robot description, xacro)
@@ -35,3 +35,10 @@
     <origin xyz="0 0 0" rpy="0 0 ${pi/2}"/>
   </joint>
+  <!-- attach tm12_tcp to gripper -->
+  <link name="tm12_tcp" />
+  <joint name="tm12_tcp_joint" type="fixed">
+    <parent link="robotiq_arg2f_base_link"/>
+    <child link="tm12_tcp"/>
+    <origin xyz="0 0 ${0.244-(0.0655/2)}" rpy="0 0 0"/>
+  </joint>
 </robot>
